File: pcb-files/keyboard/J-CH/_restore_backup_2026-06-14T18-57-00-335/J-CH.kicad_sch (KiCad schematic)
At the start: 17 parts, among them J1 JST, SW1 RST, SW2 RST, U1 STM32F072C8Tx, U2 XC6206PxxxMR-Regulator_Linear

Commit message: keyboard designed
Parts:
- C1, C3, C4, C5, C6, C7, C8, C9, R2, R3: footprint Capacitor_SMD:C_0402_1005Metric -> PCM_Capacitor_SMD_AKL:C_0402_1005Metric
- C2: footprint Capacitor_SMD:C_0603_1608Metric_Pad1.08x0.95mm_HandSolder -> PCM_Capacitor_SMD_AKL:C_0603_1608Metric_Pad1.08x0.95mm
- J1: footprint Connector_Molex:Molex_Pico-EZmate_78171-0004_1x04-1MP_P1.20mm_Vertical -> PCM_Connector_Molex:Molex_Pico-EZmate_78171-0004_1x04-1MP_P1.20mm_Vertical
- R1: footprint Resistor_SMD:R_0402_1005Metric -> PCM_Resistor_SMD_AKL:R_0402_1005Metric
- SW1, SW2: footprint Button_Switch_SMD:SW_SPST_SKQG_WithoutStem -> PCM_Button_Switch_SMD:SW_SPST_SKQG_WithoutStem
- U1: footprint Package_QFP:LQFP-48_7x7mm_P0.5mm -> PCM_Package_QFP_AKL:LQFP-48_7x7mm_P0.5mm
- U2: footprint Package_TO_SOT_SMD:SOT-23 -> PCM_Package_TO_SOT_SMD_AKL:SOT-23
Connections:
- net +3V3: no longer U1.1 (VBAT), U1.24 (VDD), U1.36 (VDDIO2), U1.48 (VDD), U1.9 (VDDA)
- net GND: no longer U1.23 (VSS), U1.35 (VSS), U1.47 (VSS), U1.8 (VSSA)
- net C1: no longer names the net of U1.21 (PB10)
- net C10: no longer names the net of U1.10 (PA0)
- net C11: no longer names the net of U1.11 (PA1)
- net C12: no longer names the net of U1.12 (PA2)
- net C13: no longer names the net of U1.13 (PA3)
- net C14: no longer names the net of U1.14 (PA4)
- net C15: no longer names the net of U1.15 (PA5)
- net C16: no longer names the net of U1.16 (PA6)
- net C17: no longer names the net of U1.17 (PA7)
- net C18: no longer names the net of U1.18 (PB0)
- net C19: no longer names the net of U1.19 (PB1)
- net C2: no longer names the net of U1.22 (PB11)
- net C3: no longer names the net of U1.37 (PA14)
- net C4: no longer names the net of U1.38 (PA15)
- net C5: no longer names the net of U1.45 (PB8)
- net C6: no longer names the net of U1.46 (PB9)
- net C7: no longer names the net of U1.4 (PC15)
- net C8: no longer names the net of U1.5 (PF0)
- net C9: no longer names the net of U1.6 (PF1)
- net R1: no longer names the net of U1.28 (PB15)
- net R2: no longer names the net of U1.27 (PB14)
- net R3: no longer names the net of U1.26 (PB13)
- net R4: no longer names the net of U1.25 (PB12)
- net R5: no longer names the net of U1.20 (PB2)
Other:
- removed sheet Switch matrix
- added sheet Untitled Sheet (untitled.kicad_sch)
